Commit message: Add real LiDAR + verified SLAM/Nav2 pipeline for Scenario B, fix two structural bugs found via live audit
This was a portfolio-grade re-audit, not a feature add: every claim below
is backed by ROS 2 topic/service introspection performed live, not assumed
or inferred from launch success.

Hard blocker fixed: the robot had no sensors at all, so slam_toolbox could
not build a real map. Added a gpu_lidar sensor on a new lidar_link
(base.xacro, mobile_manipulator.gazebo.xacro), bridged via ros_gz_bridge.
Root-caused and worked around a real sdformat limitation: gz-sim's
URDF->SDF converter silently drops the <gz_frame_id> sensor tag (confirmed
via `strings` on libgz-sensors8.so.8 + `gz sdf -p`), so /scan carries
gz-sim's auto-generated frame name instead of lidar_link -- bridged with a
zero-offset static_transform_publisher in gazebo_sim.launch.py.

Two real, structural bugs found and fixed via live introspection, not
screenshots:

1. cmd_vel message-type mismatch (the actual root cause of nearly all
   earlier "navigation doesn't work" symptoms): controller_server and
   behavior_server were publishing plain geometry_msgs/Twist while
   mobile_base_controller (diff_drive_controller) subscribes with
   TwistStamped -- a DDS type mismatch, so no Nav2-computed velocity
   command ever reached the robot regardless of what the action status
   reported. Fixed with enable_stamped_cmd_vel: true (same fix this repo
   already needed for teleop_twist_keyboard in Scenario A).

2. Costmap obstacle layer was blind: obstacle_layer.scan.max_obstacle_height
   was never set, silently defaulting to 0.0 (a per-source override distinct
   from the layer-level 2.0 default), rejecting every LiDAR point as "too
   high" since the sensor sits at z=0.20m. Confirmed via
   `ros2 service call .../get_costmap`: 0 non-zero cost cells before the
   fix, 1386 after, at world coordinates matching the real obstacle.

Also fixed: controller_server reading odometry from the wrong topic name
(/odom, zero publishers) instead of /mobile_base_controller/odom; TF
transform_tolerance widened to absorb slam_toolbox's irregular map->odom
publish timing under this CPU-constrained test environment.

Navigation reliability tuning, investigated to a precise conclusion rather
than an improved-but-vague success rate: widened progress_checker's time
budget (10s->20s) and loosened required_movement_radius (0.5->0.3) since
RegulatedPurePursuitController's correct rotate-in-place behavior was
exhausting the old budget before any translation occurred; shipped a
custom navigate_to_pose BT XML cutting a stock 5s recovery Wait action
(meant for transient dynamic obstacles this static scenario doesn't have)
to 1.0s. Measured improvement: previously-aborting goals now succeed.
The one remaining failure class was root-caused, not left vague: the
controller correctly refuses to rotate the robot's rectangular footprint
through a real inflated-cost cell near clutter (cost 0 facing forward,
cost 37 facing the goal, confirmed via get_cost_local_costmap) -- this is
safe behavior, not a bug, and "100% reliable on every goal" would require
trading away real collision-safety margin.

Added verify_scenario_b.py: an automated, 4-layer check (SLAM map content,
Nav2 lifecycle states via the real lifecycle service, TF resolution via an
actual tf2 lookup, and a real NavigateToPose goal watched for its true
terminal status) that reports ABORTED/CANCELED honestly rather than
treating "didn't crash" as success.

Also along the way: found and documented a real environment failure
(Gazebo's gz sim process silently died after ~80 minutes in GUI mode while
Nav2/SLAM/robot_state_publisher kept running orphaned) and distinguished
it from actual config bugs by checking `ps -ef`, not assuming from
symptoms alone.

Docs (docs/TESTING.md, SCENARIOS.md, README.md) updated with the full
evidence trail -- root causes, exact commands, before/after measurements
-- and two screenshots (Gazebo physics + RViz showing the live SLAM map
and real LaserScan hits) replacing the prior "partial, unverified"
Scenario B status. Roadmap updated: LiDAR/SLAM item marked done, static-map
item replaced with the inflation-radius/reachability tradeoff this
investigation actually surfaced.

Co-Authored-By: Claude Sonnet 4.6 <noreply@anthropic.com>

File: src/mobile_manipulator_description/urdf/base.xacro (robot description, xacro)
@@ -80,3 +80,30 @@
   <xacro:wheel prefix="rear_left"   x_reflect="-1" y_reflect="1"/>
   <xacro:wheel prefix="rear_right"  x_reflect="-1" y_reflect="-1"/>
+  <!-- ###################################################################
+       2D LiDAR for Scenario B (Nav2 + SLAM). Previously absent entirely
+       (confirmed in the forensic audit and documented as a known gap in
+       docs/TESTING.md / SCENARIOS.md): slam_toolbox cannot build a real
+       map without range data, so this was a hard blocker for any genuine
+       SLAM/navigation claim, not just a nice-to-have. Mounted at the
+       front of the base (x=-0.30), opposite the arm mount (x=+0.20,
+       see arm.xacro) to minimize self-occlusion of the scan by the arm.
+       ################################################################### -->
+  <link name="lidar_link">
+    <inertial>
+      <mass value="0.15"/>
+      <inertia ixx="0.0001" ixy="0" ixz="0" iyy="0.0001" iyz="0" izz="0.0001"/>
+    </inertial>
+    <visual>
+      <geometry><cylinder radius="0.04" length="0.05"/></geometry>
+      <material name="chassis_grey"/>
+    </visual>
+    <collision>
+      <geometry><cylinder radius="0.04" length="0.05"/></geometry>
+    </collision>
+  </link>
+  <joint name="lidar_joint" type="fixed">
+    <parent link="base_link"/>
+    <child link="lidar_link"/>
+    <origin xyz="-0.30 0.0 0.20" rpy="0 0 0"/>
+  </joint>
 </robot>

File: src/mobile_manipulator_gazebo/urdf/mobile_manipulator.gazebo.xacro (robot description, xacro)
@@ -28,22 +28,58 @@
     </plugin>
   </gazebo>
-  <!-- #################### Perception roadmap hooks ####################
-       No sensors exist on the robot yet (confirmed in the forensic audit:
-       README claimed cameras/LiDAR, code had none). These are commented
-       placeholders showing exactly where perception attaches once a
-       sensor mount is added to base.xacro. Not enabled by default, so
-       this package keeps building/launching cleanly without sensor
-       plugins that have no corresponding link. Plugin names below use
-       the Gazebo Sim (gz-sim) sensor system, not Gazebo Classic.
-  <gazebo reference="camera_link">
-    <sensor type="camera" name="rgb_camera">
-      <plugin filename="gz-sim-sensors-system" name="gz::sim::systems::Sensors"/>
+  <!-- ###################################################################
+       LiDAR sensor (Scenario B / Nav2 + SLAM). Real, not a placeholder:
+       a `lidar_link` now exists in base.xacro (mounted at the base
+       front), so this sensor block is enabled by default. Topic is
+       `/scan` directly (not `/perception/scan`) to match what
+       mobile_manipulator_bringup/config/nav2_params.yaml's costmaps and
+       slam_toolbox both expect out of the box: no remap needed.
+       The world-level `gz-sim-sensors-system` plugin (already loaded in
+       mobile_manipulator_world.world) is what actually runs this sensor;
+       this block only declares it on the link.
+       ################################################################### -->
+  <gazebo reference="lidar_link">
+    <sensor type="gpu_lidar" name="lidar">
+      <topic>/scan</topic>
+      <!-- AUDIT FIX: gz-sim stamps the published LaserScan with its own
+           auto-generated scoped frame ("mobile_manipulator/base_link/lidar"),
+           not "lidar_link", the frame robot_state_publisher actually
+           publishes via TF. Nav2's costmap and slam_toolbox both call tf2
+           lookupTransform() using the scan message's frame_id, so an
+           unmatched frame_id silently breaks both with no Gazebo-side
+           error. Tried fixing it here with a `<gz_frame_id>lidar_link</gz_frame_id>`
+           element (confirmed to be the right keyword by `strings` on
+           libgz-sensors8.so.8); verified by an actual run that
+           sdformat's URDF->SDF converter silently drops it before the
+           sensor ever sees it (`gz_frame_id` is not a recognized SDF
+           schema element for <sensor>, unlike <ros2_control>, which has
+           explicit pass-through support). Fixed instead with a static
+           transform publisher bridging the two frame names in
+           gazebo_sim.launch.py, since they are physically coincident. -->
+      <update_rate>10</update_rate>
+      <always_on>true</always_on>
+      <visualize>true</visualize>
+      <lidar>
+        <scan>
+          <horizontal>
+            <samples>360</samples>
+            <resolution>1</resolution>
+            <min_angle>-3.14159</min_angle>
+            <max_angle>3.14159</max_angle>
+          </horizontal>
+        </scan>
+        <range>
+          <min>0.12</min>
+          <max>12.0</max>
+          <resolution>0.01</resolution>
+        </range>
+      </lidar>
     </sensor>
   </gazebo>
-  <gazebo reference="lidar_link">
-    <sensor type="gpu_lidar" name="lidar">
-      <topic>/perception/scan</topic>
-      <update_rate>10</update_rate>
-    </sensor>
+  <!-- #################### Perception roadmap hook (camera) ############
+       Camera still genuinely absent: no camera_link exists in
+       base.xacro/arm.xacro. Left as a placeholder; not enabled.
+  <gazebo reference="camera_link">
+    <sensor type="camera" name="rgb_camera"/>
   </gazebo>
   ##################################################################### -->
